File: Schematics/Reflow.kicad_pcb (KiCad board)
At the start: 2 copper layers, 1 part

Commit message: Finally completed V1 control board
Parts:
- added C1: 100nF, Capacitor_SMD:C_0805_2012Metric, B.Cu at (207.3, 94.7)
- added C10: 1.5pF, Capacitor_SMD:C_0805_2012Metric, B.Cu at (216.5, 81.8)
- added C11: 1uF, Capacitor_SMD:C_0805_2012Metric, B.Cu at (180.1, 123.8)
- added C12: 1uF, Capacitor_SMD:C_0805_2012Metric, B.Cu at (180.3, 107.8)
- added C2: 1uF, Capacitor_SMD:C_0805_2012Metric, B.Cu at (207.2, 91.5)
- added C3: 100nF, Capacitor_SMD:C_0805_2012Metric, B.Cu at (207.1, 72.5)
- added C4: 4.7uF, Capacitor_SMD:C_0805_2012Metric, B.Cu at (207.1, 75.7)
- added C5: 100nF, Capacitor_SMD:C_0805_2012Metric, B.Cu at (199.0, 67.7)
- added C6: 4.7uF, Capacitor_SMD:C_0805_2012Metric, B.Cu at (190.7, 96.9)
- added C7: 20pF, Capacitor_SMD:C_0805_2012Metric, B.Cu at (216.5, 85.3)
- added C8: 20pF, Capacitor_SMD:C_0805_2012Metric, B.Cu at (216.6, 88.6)
- added C9: 1.5pF, Capacitor_SMD:C_0805_2012Metric, B.Cu at (216.6, 78.7)
- added CN1: 100nF, Resistor_SMD:R_Array_Convex_4x0603, B.Cu at (182.0, 83.4)
- added D1: LED, LED_SMD:LED_0805_2012Metric, F.Cu at (203.4, 67.7)
- added D2: LED, LED_SMD:LED_0805_2012Metric, F.Cu at (223.8, 67.7)
- added D3: LED, LED_SMD:LED_0805_2012Metric, F.Cu at (182.9, 214.4)
- added D4: LED, LED_SMD:LED_0805_2012Metric, F.Cu at (206.7, 200.9)
- added D5: LED, LED_SMD:LED_0805_2012Metric, F.Cu at (206.7, 228.1)
- added G***: LOGO, LOGO, F.Cu at (197.2, 149.4)
- added J1: USB_C_Receptacle, Reflow:Jing_USB-C_Vert_C168703, F.Cu at (177.8, 76.4)
- added J2: Conn_01x02, Reflow:Connector_1x02_5mm, F.Cu at (194.7, 243.7)
- added J3: Conn_01x10, Connector_PinHeader_2.54mm:PinHeader_1x10_P2.54mm_Vertical, F.Cu at (182.1, 187.6)
- added J4: Conn_01x12, Reflow:A2501WR-12P1-Conn, F.Cu at (175.5, 222.7)
- added J5: Conn_01x04, Connector_PinHeader_2.54mm:PinHeader_1x04_P2.54mm_Vertical, F.Cu at (191.1, 235.4)
- added J6: Prog, Connector_PinHeader_2.54mm:PinHeader_1x06_P2.54mm_Vertical, F.Cu at (200.7, 72.8)
- added J7: BreadboardPwr, Connector_PinHeader_2.54mm:PinHeader_1x02_P2.54mm_Vertical, F.Cu at (226.6, 84.0)
- added J8: Conn_01x03, Connector_PinHeader_2.54mm:PinHeader_1x03_P2.54mm_Vertical, F.Cu at (217.1, 212.0)
- added J9: Conn_01x04, Connector_PinHeader_2.54mm:PinHeader_1x04_P2.54mm_Vertical, F.Cu at (194.3, 114.2)
- added L1: L_Small, Inductor_SMD:L_0603_1608Metric, B.Cu at (207.3, 97.9)
- added R1: 0, Resistor_SMD:R_0805_2012Metric, B.Cu at (207.1, 85.2)
- added R2: 0, Resistor_SMD:R_0805_2012Metric, B.Cu at (207.2, 88.3)
- added R3: 0, Resistor_SMD:R_0805_2012Metric, B.Cu at (207.1, 78.9)
- added R4: 0, Resistor_SMD:R_0805_2012Metric, B.Cu at (207.1, 82.1)
- added REF**: Pin_D1.0mm_L10.0mm, Connector_Pin:Pin_D1.0mm_L10.0mm, F.Cu at (175.8, 192.6)
- added REF**: Pin_D1.0mm_L10.0mm, Connector_Pin:Pin_D1.0mm_L10.0mm, F.Cu at (221.3, 192.6)
- added REF**: Pin_D1.0mm_L10.0mm, Connector_Pin:Pin_D1.0mm_L10.0mm, F.Cu at (192.6, 68.5)
- added REF**: Pin_D1.0mm_L10.0mm, Connector_Pin:Pin_D1.0mm_L10.0mm, F.Cu at (180.8, 243.1)
- added REF**: Pin_D1.0mm_L10.0mm, Connector_Pin:Pin_D1.0mm_L10.0mm, F.Cu at (226.2, 233.1)
- added RN1: 1k, Resistor_SMD:R_Array_Convex_4x0603, F.Cu at (178.6, 69.3)
- added RN2: R_Pack04, Resistor_SMD:R_Array_Convex_4x0603, B.Cu at (214.8, 104.3)
- added RN3: R_Pack04, Resistor_SMD:R_Array_Convex_4x0603, F.Cu at (214.1, 58.0)
- added RN4: R_Pack04, Resistor_SMD:R_Array_Convex_4x0603, F.Cu at (195.2, 229.4)
- added Ref**: Val**, NFCBuisness:W, F.Cu at (172.0, 244.8)
- added SW1: SW_Push, Button_Switch_SMD:SW_Push_1P1T_NO_6x6mm_H9.5mm, F.Cu at (178.2, 57.1)
- added SW2: SW_Push, Button_Switch_SMD:SW_Push_1P1T_NO_6x6mm_H9.5mm, F.Cu at (213.8, 67.6)
- added SW4: SW_Push, Button_Switch_SMD:SW_Push_1P1T_NO_6x6mm_H9.5mm, F.Cu at (220.1, 176.4)
- added SW5: SW_Push, Button_Switch_SMD:SW_Push_1P1T_NO_6x6mm_H9.5mm, F.Cu at (177.8, 176.2)
- added SW6: SW_Push, Button_Switch_SMD:SW_Push_1P1T_NO_6x6mm_H9.5mm, F.Cu at (198.8, 176.2)
- added SW7: Rotary_Encoder, Reflow:Circular_Rotary_Enc, F.Cu at (198.8, 214.3)
- added SW8: SW_Push, Button_Switch_SMD:SW_Push_1P1T_NO_6x6mm_H9.5mm, F.Cu at (198.8, 214.3)
- added U1: MCP9600, Package_DFN_QFN:QFN-20-1EP_5x5mm_P0.65mm_EP3.35x3.35mm, B.Cu at (215.3, 229.4)
- added U2: STM32F411RETx, Package_QFP:LQFP-64_10x10mm_P0.5mm, B.Cu at (195.4, 84.7)
- added U3: TLV1117-33, Package_TO_SOT_SMD:SOT-223-3_TabPin2, B.Cu at (178.7, 115.6)
- added Y1: 8MHz, Crystal:Crystal_SMD_SeikoEpson_TSX3225-4Pin_3.2x2.5mm, B.Cu at (212.0, 86.5)
- added Y2: 32.768kHz, Crystal:Crystal_SMD_3215-2Pin_3.2x1.5mm, B.Cu at (212.2, 80.5)
Routing:
- net VCC: track 0.00 -> 351.5 mm, vias 0 -> 4
- net SDA: track 0.00 -> 205.8 mm, vias 0 -> 6
- net SCL: track 0.00 -> 195.5 mm, vias 0 -> 6
- net Alert3: track 0.00 -> 169.0 mm, vias 0 -> 2
- net Alert4: track 0.00 -> 168.8 mm, vias 0 -> 2
- net +5V: track 0.00 -> 161.0 mm, vias 0 -> 2
- net DOWN: track 0.00 -> 153.1 mm, vias 0 -> 1
- net EncC: track 0.00 -> 148.4 mm, vias 0 -> 1
- net LED3: track 0.00 -> 146.3 mm, vias 0 -> 1
- net LED5: track 0.00 -> 145.3 mm, vias 0 -> 1
- net SW7-StartStop: track 0.00 -> 139.0 mm, vias 0 -> 3
- net UP: track 0.00 -> 135.0 mm, vias 0 -> 1
- net SW5-Function: track 0.00 -> 122.6 mm, vias 0 -> 1
- net LED4: track 0.00 -> 122.1 mm, vias 0 -> 1
- net LowCtrl: track 0.00 -> 109.1 mm, vias 0 -> 1
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- added copper zone on B.Cu, net VSS
- added copper zone on F.Cu, net VSS
Other:
- board outline added: 64.4 x 196.6 mm
- board text added: "+5v Gnd +12V High Low ROT FAN Lamp Temp1 Temp2 Safe Zero"
- board text added: "@RMA_Electronics"
- board text added: "Easy Circuit Bake Oven"
- board text added: "High HighCtrl Low LowCtrl ROT RotCtrl Fan FanCtrl Lamp LampCtrl"
- board text added: "V1"
