File: Schematics/Reflow.sch (KiCad schematic (older format))
At the start: 36 parts

Commit message: Finally completed V1 control board
Parts:
- removed C? (x5): 0.1uF, symbol Device:C_Small
- removed J?: Conn_01x12, symbol Connector_Generic:Conn_01x12
- removed J?: USB_B_Mini, symbol badge-cache:USB_B_Mini
- removed J?: Conn_01x40, symbol Connector_Generic:Conn_01x40
- removed J? (x2): Conn_01x11, symbol Connector_Generic:Conn_01x11
- removed J?: Conn_01x02, symbol Connector_Generic:Conn_01x02
- removed R? (x5): R_Small, symbol Device:R_Small
- removed R?: 10k, symbol Device:R_Small
- removed U?: badge-rescue_ESP32-WROOM, ESP32-footprints-Lib:ESP32-WROOM, symbol badge-cache:badge-rescue_ESP32-WROOM
- removed U?: otter_CH330, symbol badge-cache:badge-rescue_otter_CH330-CH330-cache
- added C1, C3, C5: 100nF, Capacitor_SMD:C_0805_2012Metric, symbol Device:C_Small
- added C10, C9: 1.5pF, Capacitor_SMD:C_0805_2012Metric, symbol Device:C_Small
- added C2: 1uF, Capacitor_SMD:C_0805_2012Metric, symbol Device:C_Small
- added C4, C6: 4.7uF, Capacitor_SMD:C_0805_2012Metric, symbol Device:C_Small
- added C7, C8: 20pF, Capacitor_SMD:C_0805_2012Metric, symbol Device:C_Small
- added CN1: 100nF, Resistor_SMD:R_Array_Convex_4x0603, symbol Device:R_Pack04
- added J1: USB_C_Receptacle, Reflow:Jing_USB-C_Vert_C168703, symbol Connector:USB_C_Receptacle
- added J2: Conn_01x02, Reflow:Connector_1x02_5mm, symbol Connector_Generic:Conn_01x02
- added J3: Conn_01x10, Connector_PinHeader_2.54mm:PinHeader_1x10_P2.54mm_Vertical, symbol Connector_Generic:Conn_01x10
- added J5, J9: Conn_01x04, Connector_PinHeader_2.54mm:PinHeader_1x04_P2.54mm_Vertical, symbol Connector_Generic:Conn_01x04
- added J6: Prog, Connector_PinHeader_2.54mm:PinHeader_1x06_P2.54mm_Vertical, symbol Connector_Generic:Conn_01x06
- added J7: BreadboardPwr, Connector_PinHeader_2.54mm:PinHeader_1x02_P2.54mm_Vertical, symbol Connector_Generic:Conn_01x02
- added J8: Conn_01x03, Connector_PinHeader_2.54mm:PinHeader_1x03_P2.54mm_Vertical, symbol Connector_Generic:Conn_01x03
- added L1: L_Small, Inductor_SMD:L_0603_1608Metric, symbol Device:L_Small
- added R1, R2, R3, R4: 0, Resistor_SMD:R_0805_2012Metric, symbol Device:R_Small
- added RN1: 1k, Resistor_SMD:R_Array_Convex_4x0603, symbol Device:R_Pack04
- added RN2, RN3, RN4: R_Pack04, Resistor_SMD:R_Array_Convex_4x0603, symbol Device:R_Pack04
- added U1: MCP9600, Package_DFN_QFN:QFN-20-1EP_5x5mm_P0.65mm_EP3.35x3.35mm, symbol Reflow:MCP9600
- added U2: STM32F411RETx, Package_QFP:LQFP-64_10x10mm_P0.5mm, symbol MCU_ST_STM32F4:STM32F411RETx
- added Y1: 8MHz, Crystal:Crystal_SMD_SeikoEpson_TSX3225-4Pin_3.2x2.5mm, symbol Device:Crystal_GND24
- added Y2: 32.768kHz, Crystal:Crystal_SMD_3215-2Pin_3.2x1.5mm, symbol Device:Crystal_Small
- C11, C12: renamed from C?; footprint (none) -> Capacitor_SMD:C_0805_2012Metric
- D1, D2, D3, D4, D5: renamed from D?; footprint (none) -> LED_SMD:LED_0805_2012Metric
- J4: renamed from J?; footprint (none) -> Reflow:A2501WR-12P1-Conn
- SW1, SW2, SW3, SW4, SW5, SW6, SW8: renamed from SW?; footprint (none) -> Button_Switch_SMD:SW_Push_1P1T_NO_6x6mm_H9.5mm
- SW7: renamed from SW?; footprint (none) -> Reflow:Circular_Rotary_Enc
- U3: renamed from U?; footprint (none) -> Package_TO_SOT_SMD:SOT-223-3_TabPin2; symbol badge-cache:TLV1117-33 -> Reflow-rescue:TLV1117-33-badge-cache
Connections:
- net +5V: now also J1.A4 (VBUS), J1.A9 (VBUS), J1.B4 (VBUS), J1.B9 (VBUS)
- net DOWN: now also J8.3 (Pin_3), U2.38 (PC7)
- net FAN: now also J3.7 (Pin_7)
- net HI: now also J3.1 (Pin_1)
- net LAMP: now also J3.9 (Pin_9)
- net LED1: now also D1.2 (A), U2.8 (PC0); no longer D1.1 (K)
- net LED2: now also D2.2 (A), U2.9 (PC1); no longer D2.1 (K)
- net LED3: now also D3.2 (A), U2.10 (PC2); no longer D3.1 (K)
- net LED4: now also D4.2 (A), U2.11 (PC3); no longer D4.1 (K)
- net LED5: now also D5.2 (A), U2.24 (PC4); no longer D5.1 (K)
- net LOW: now also J3.3 (Pin_3)
- net ROT: now also J3.5 (Pin_5)
- net RX: now also U2.42 (PA9)
- net SW1-Preheat: now also U2.14 (PA0)
- net SW2-ECO: now also U2.15 (PA1)
- net SW3-Convection: now also U2.16 (PA2)
- net SW4-Temp: now also U2.17 (PA3)
- net SW5-Function: now also U2.36 (PB15)
- net SW6-Time: now also U2.21 (PA5)
- net SW7-StartStop: now also U2.22 (PA6)
- net TX: now also U2.43 (PA10)
- net Temp1: now also J5.1 (Pin_1)
- net Temp2: now also J5.3 (Pin_3)
- net UP: now also J8.1 (Pin_1), U2.25 (PC5)
- net VCC: now also C3.1, C4.1, CN1.5 (R4.2), CN1.6 (R3.2), CN1.7 (R2.2), CN1.8 (R1.2), J6.6 (Pin_6), J7.1 (Pin_1), J9.2 (Pin_2), L1.2, RN2.1 (R1.1), RN2.2 (R2.1), U1.8 (VDD), U2.1 (VBAT), U2.19 (VDD), U2.32 (VDD), U2.48 (VDD), U2.64 (VDD)
- net VSS: now also J4.2 (Pin_2), SW1.1, SW2.1, SW3.1, SW4.1, SW5.1, SW6.1, SW8.1, C1.2, C10.2, C2.2, C3.2, C4.2, C5.1, C6.2, C7.2, C8.2, C9.2, CN1.1 (R1.1), CN1.2 (R2.1), CN1.3 (R3.1), CN1.4 (R4.1), J1.A1 (GND), J1.A12 (GND), J1.B1 (GND), J1.B12 (GND), J1.S1 (SHIELD), J6.5 (Pin_5), J7.2 (Pin_2), J9.1 (Pin_1), RN1.7 (R2.2), RN1.8 (R1.2), RN3.1 (R1.1), RN3.2 (R2.1), RN3.3 (R3.1), RN3.4 (R4.1), RN4.1 (R1.1), RN4.2 (R2.1), RN4.3 (R3.1), RN4.4 (R4.1), U1.1 (GND), U1.10 (GND), U1.13 (GND), U1.16 (ADDR), U1.17 (GND), U1.18 (GND), U1.21 (GND_EP), U1.3 (GND), U1.5 (GND), U1.6 (GND), U1.7 (GND), U1.9 (GND), U2.12 (VSSA), U2.18 (VSS), U2.31 (VSS), U2.47 (VSS), U2.63 (VSS), Y1.2, Y1.4
- removed net GND: J4.2 (Pin_2), SW1.1, SW2.1, SW3.1, SW4.1, SW5.1, SW6.1, SW7.C, SW8.1
- new net: D1.1 (K), RN3.7 (R2.2)
- new net: D2.1 (K), RN3.8 (R1.2)
- new net: D3.1 (K), RN4.8 (R1.2)
- new net: D4.1 (K), RN4.7 (R2.2)
- new net: D5.1 (K), RN4.6 (R3.2)
- new net: R3.1, U2.3 (PC14)
- new net: C6.1, U2.30 (VCAP1)
- new net: R4.1, U2.4 (PC15)
- new net: R1.1, U2.5 (PH0)
- new net: R2.1, U2.6 (PH1)
- new net: C7.1, R1.2, Y1.1
- new net: C8.1, R2.2, Y1.3
- new net: C9.1, R3.2, Y2.1
- new net: C10.1, R4.2, Y2.2
- new net: J1.A5 (CC1), RN1.2 (R2.1)
- new net: J1.B5 (CC2), RN1.1 (R1.1)
- new net Alert1: U1.11 (Alert_1)
- new net Alert2: U1.12 (Alert_2)
- new net Alert3: U1.14 (Alert_3), U2.51 (PC10)
- new net Alert4: U1.15 (Alert_4), U2.52 (PC11)
- new net Boot0: J6.2 (Pin_2), U2.60 (BOOT0)
- new net D+: J1.A6 (D+), J1.B6 (D+), U2.45 (PA12)
- new net D-: J1.A7 (D-), J1.B7 (D-), U2.44 (PA11)
- new net EncC: J8.2 (Pin_2), SW7.C, U2.37 (PC6)
- new net FanCtrl: J3.8 (Pin_8)
- new net HighCtrl: J3.2 (Pin_2), U2.41 (PA8)
- new net LampCtrl: J3.10 (Pin_10)
- new net LowCtrl: J3.4 (Pin_4), U2.40 (PC9)
- new net RST: C5.2, J6.1 (Pin_1), U2.7 (NRST)
- new net RotCtrl: J3.6 (Pin_6)
- new net SCL: J9.4 (Pin_4), RN2.8 (R1.2), U1.19 (SCL), U2.58 (PB6)
- new net SDA: J9.3 (Pin_3), RN2.7 (R2.2), U1.20 (SDA), U2.59 (PB7)
- new net SWCLK: J6.3 (Pin_3), U2.49 (PA14)
- new net SWDIO: J6.4 (Pin_4), U2.46 (PA13)
- new net Temp1out: J2.1 (Pin_1), J5.2 (Pin_2), U1.4 (Vin-)
- new net Temp2out: J2.2 (Pin_2), J5.4 (Pin_4), U1.2 (Vin+)
- new net VDDA: C1.1, C2.1, L1.1, U2.13 (VDDA)
- no-connect marks 9 -> 23
Other:
- note removed: "Active Low"
- moved on the sheet: C11, C12, D1, D2, D3, D4, D5, J4, SW1, SW2, SW3, SW4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
